Commit message: Configuing bimanual kuka for cuRobo setup

File: urdf/dual_arm/dual_arm_w_grippers.urdf (robot description, URDF)
Before this commit: robot bh_robot, 39 links, 38 joints
Links:
- link left_camera: geometry collision box size=0.025 0.090 0.025; visual mesh filename=package://kuka_maniskill_sim/meshes/camera/d435.dae
- link right_camera: geometry collision box size=0.025 0.090 0.025; visual mesh filename=package://kuka_maniskill_sim/meshes/camera/d435.dae

Commit message: Adjusted ee_link orientation by 90 degrees Adjusted camera position Removed unnessesary comments

File: urdf/dual_arm/dual_arm_w_grippers.urdf (robot description, URDF)
Before this commit: robot bh_robot, 39 links, 38 joints
Joints:
- joint left_arm_joint_ee: origin xyz=0 0 0.035 rpy=0 0 0 -> xyz=0 0 0.035 rpy=0 0 1.57
- joint left_camera_joint: origin xyz=0.07 0.032 0.065 rpy=0 0 0 -> xyz=0.08 0.032 0.03 rpy=0 0 0
- joint right_arm_joint_ee: origin xyz=0 0 0.035 rpy=0 0 0 -> xyz=0 0 0.035 rpy=0 0 1.57
- joint right_camera_joint: origin xyz=0.07 0.032 0.065 rpy=0 0 0 -> xyz=0.08 0.032 0.03 rpy=0 0 0

Commit message: Fixed collision support for gripper

File: urdf/dual_arm/dual_arm_w_grippers.urdf (robot description, URDF)
Before this commit: robot bh_robot, 39 links, 38 joints
Links:
- link left_robotiq_hande_left_finger: mass None -> 0.03804; geometry collision mesh filename=kuka_maniskill_sim/meshes/gripper/finger_collision.dae; visual mesh filename=kuka_maniskill_sim/meshes/gripper/finger.dae
- link left_robotiq_hande_link: mass None -> 0.86387; geometry collision mesh filename=kuka_maniskill_sim/meshes/gripper/hande.dae; visual mesh filename=kuka_maniskill_sim/meshes/gripper/hande.dae
- link left_robotiq_hande_right_finger: mass None -> 0.03804; geometry collision mesh filename=kuka_maniskill_sim/meshes/gripper/finger_collision.dae; visual mesh filename=kuka_maniskill_sim/meshes/gripper/finger.dae
- link right_robotiq_hande_left_finger: mass None -> 0.03804; geometry collision mesh filename=kuka_maniskill_sim/meshes/gripper/finger_collision.dae; visual mesh filename=kuka_maniskill_sim/meshes/gripper/finger.dae
- link right_robotiq_hande_link: mass None -> 0.86387; geometry collision mesh filename=kuka_maniskill_sim/meshes/gripper/hande.dae; visual mesh filename=kuka_maniskill_sim/meshes/gripper/hande.dae
- link right_robotiq_hande_right_finger: mass None -> 0.03804; geometry collision mesh filename=kuka_maniskill_sim/meshes/gripper/finger_collision.dae; visual mesh filename=kuka_maniskill_sim/meshes/gripper/finger.dae
Joints:
- joint left_robotiq_hande_left_finger_joint: limit lower=0.0 upper=0.03 effort=130 velocity=0.15 -> lower=0.0 upper=0.025 effort=130 velocity=0.15
- joint left_robotiq_hande_right_finger_joint: limit lower=0.0 upper=0.03 effort=130 velocity=0.15 -> lower=0.0 upper=0.025 effort=130 velocity=0.15; mimic joint=left_robotiq_hande_left_finger_joint multiplier=1 offset=0 -> (none)
- joint right_robotiq_hande_left_finger_joint: limit lower=0.0 upper=0.03 effort=130 velocity=0.15 -> lower=0.0 upper=0.025 effort=130 velocity=0.15
- joint right_robotiq_hande_right_finger_joint: limit lower=0.0 upper=0.03 effort=130 velocity=0.15 -> lower=0.0 upper=0.025 effort=130 velocity=0.15; mimic joint=right_robotiq_hande_left_finger_joint multiplier=1 offset=0 -> (none)

Commit message: fixed wrist camera views

File: urdf/dual_arm/dual_arm_w_grippers.urdf (robot description, URDF)
Before this commit: robot bh_robot, 39 links, 38 joints
Joints:
- joint left_camera_joint: origin xyz=0.08 0.032 0.03 rpy=0 0 0 -> xyz=0.08 0.0 0.03 rpy=0 -1.57 3.141592653589793
- joint right_camera_joint: origin xyz=0.08 0.032 0.03 rpy=0 0 0 -> xyz=0.08 0.0 0.03 rpy=0 -1.57 3.141592653589793

Commit message: - Adjusted joint limits - Artificially increased gripper openning width

File: urdf/dual_arm/dual_arm_w_grippers.urdf (robot description, URDF)
Before this commit: robot bh_robot, 39 links, 38 joints
Joints:
- joint left_arm_A1: limit lower=-2.9670597283903604 upper=2.9670597283903604 effort=200 velocity=1.710422666954443 -> lower=-3.14159265359 upper=3.14159265359 effort=200 velocity=1.710422666954443
- joint left_arm_A2: limit lower=-2.0943951023931953 upper=2.0943951023931953 effort=200 velocity=1.710422666954443 -> lower=-3.14159265359 upper=3.14159265359 effort=200 velocity=1.710422666954443
- joint left_arm_A3: limit lower=-2.9670597283903604 upper=2.9670597283903604 effort=200 velocity=1.7453292519943295 -> lower=-3.14159265359 upper=3.14159265359 effort=200 velocity=1.7453292519943295
- joint left_arm_A4: limit lower=-2.0943951023931953 upper=2.0943951023931953 effort=200 velocity=2.2689280275926285 -> lower=-3.14159265359 upper=3.14159265359 effort=200 velocity=2.2689280275926285
- joint left_arm_A5: limit lower=-2.9670597283903604 upper=2.9670597283903604 effort=200 velocity=2.443460952792061 -> lower=-3.14159265359 upper=3.14159265359 effort=200 velocity=2.443460952792061
- joint left_arm_A6: limit lower=-2.0943951023931953 upper=2.0943951023931953 effort=200 velocity=3.141592653589793 -> lower=-3.14159265359 upper=3.14159265359 effort=200 velocity=3.141592653589793
- joint left_arm_A7: limit lower=-3.0543261909900763 upper=3.0543261909900763 effort=200 velocity=3.141592653589793 -> lower=-3.14159265359 upper=3.14159265359 effort=200 velocity=3.141592653589793
- joint left_robotiq_hande_left_finger_joint: limit lower=0.0 upper=0.025 effort=130 velocity=0.15 -> lower=0.0 upper=0.0425 effort=130 velocity=0.15
- joint left_robotiq_hande_right_finger_joint: limit lower=0.0 upper=0.025 effort=130 velocity=0.15 -> lower=0.0 upper=0.0425 effort=130 velocity=0.15
- joint right_arm_A1: limit lower=-2.9670597283903604 upper=2.9670597283903604 effort=200 velocity=1.710422666954443 -> lower=-3.14159265359 upper=3.14159265359 effort=200 velocity=1.710422666954443
- joint right_arm_A2: limit lower=-2.0943951023931953 upper=2.0943951023931953 effort=200 velocity=1.710422666954443 -> lower=-3.14159265359 upper=3.14159265359 effort=200 velocity=1.710422666954443
- joint right_arm_A3: limit lower=-2.9670597283903604 upper=2.9670597283903604 effort=200 velocity=1.7453292519943295 -> lower=-3.14159265359 upper=3.14159265359 effort=200 velocity=1.7453292519943295
- joint right_arm_A4: limit lower=-2.0943951023931953 upper=2.0943951023931953 effort=200 velocity=2.2689280275926285 -> lower=-3.14159265359 upper=3.14159265359 effort=200 velocity=2.2689280275926285
- joint right_arm_A5: limit lower=-2.9670597283903604 upper=2.9670597283903604 effort=200 velocity=2.443460952792061 -> lower=-3.14159265359 upper=3.14159265359 effort=200 velocity=2.443460952792061
- joint right_arm_A6: limit lower=-2.0943951023931953 upper=2.0943951023931953 effort=200 velocity=3.141592653589793 -> lower=-3.14159265359 upper=3.14159265359 effort=200 velocity=3.141592653589793
- joint right_arm_A7: limit lower=-3.0543261909900763 upper=3.0543261909900763 effort=200 velocity=3.141592653589793 -> lower=-3.14159265359 upper=3.14159265359 effort=200 velocity=3.141592653589793
- joint right_robotiq_hande_left_finger_joint: limit lower=0.0 upper=0.025 effort=130 velocity=0.15 -> lower=0.0 upper=0.0425 effort=130 velocity=0.15
- joint right_robotiq_hande_right_finger_joint: limit lower=0.0 upper=0.025 effort=130 velocity=0.15 -> lower=0.0 upper=0.0425 effort=130 velocity=0.15

Commit message: Matchhing real robot config

File: urdf/dual_arm/dual_arm_w_grippers.urdf (robot description, URDF)
Before this commit: robot bh_robot, 39 links, 38 joints
Joints:
- joint left_gripper_weld: origin xyz=0 0 0 rpy=0 0 0 -> xyz=0 0 0 rpy=0 0 -1.57; parent left_arm_link_7 -> left_arm_link_ee
- joint right_gripper_weld: origin xyz=0 0 0 rpy=0 0 0 -> xyz=0 0 0 rpy=0 0 -1.57; parent right_arm_link_7 -> right_arm_link_ee

Commit message: adjusted camera views

File: urdf/dual_arm/dual_arm_w_grippers.urdf (robot description, URDF)
Before this commit: robot bh_robot, 39 links, 38 joints
Joints:
- joint left_camera_joint: origin xyz=0.08 0.0 0.03 rpy=0 -1.57 3.141592653589793 -> xyz=0.08 0.0 0.03 rpy=0 -1.2 3.141592653589793
- joint right_camera_joint: origin xyz=0.08 0.0 0.03 rpy=0 -1.57 3.141592653589793 -> xyz=0.08 0.0 0.03 rpy=0 -1.2 3.141592653589793
